Commit message: flexible parameterized urdf

File: velodyne_description/urdf/VLP-16-namespacing.urdf.xacro (robot description, xacro)
@@ -2,11 +2,11 @@
 <robot xmlns:xacro="http://www.ros.org/wiki/xacro" name="VLP-16">
   <xacro:property name="M_PI" value="3.1415926535897931" />
-  <xacro:macro name="VLP-16" params="*origin parent:=base_link name:=velodyne topic:=/velodyne_points hz:=10 lasers:=16 samples:=1875 collision_range:=0.3 min_range:=0.9 max_range:=130.0 noise:=0.008 min_angle:=-${M_PI} max_angle:=${M_PI}">
-    <joint name="${name}_base_mount_joint" type="fixed">
+  <xacro:macro name="VLP-16" params="*origin namespace parent:=base_link name:=velodyne topic:=velodyne_points hz:=10 lasers:=16 samples:=1875 collision_range:=0.3 min_range:=0.9 max_range:=130.0 noise:=0.008 min_angle:=-${M_PI} max_angle:=${M_PI}">
+    <joint name="${namespace}/${name}_base_mount_joint" type="fixed">
       <xacro:insert_block name="origin" />
-      <parent link="${parent}"/>
-      <child link="${name}_base_link"/>
+      <parent link="${namespace}/${parent}"/>
+      <child link="${namespace}/${name}_base_link"/>
     </joint>
-    <link name="${name}_base_link">
+    <link name="${namespace}/${name}_base_link">
       <inertial>
         <mass value="0.03"/>
@@ -33,10 +33,10 @@
       </collision>
     </link>
-    <joint name="${name}_base_scan_joint" type="fixed" >
+    <joint name="${namespace}/${name}_base_scan_joint" type="fixed" >
       <origin xyz="0 0 0.0377" rpy="0 0 0" />
-      <parent link="${name}_base_link" />
-      <child link="${name}"/>
+      <parent link="${namespace}/${name}_base_link" />
+      <child link="${namespace}/${name}"/>
     </joint>
-    <link name="${name}">
+    <link name="${namespace}/${name}">
       <inertial>
         <mass value="0.01"/>
@@ -52,6 +52,6 @@
     </link>
     <!-- Gazebo requires the velodyne_gazebo_plugins package -->
-    <gazebo reference="${name}">
-      <sensor type="ray" name="${name}-VLP16">
+    <gazebo reference="${namespace}/${name}">
+      <sensor type="ray" name="${namespace}/${name}-VLP16">
         <pose>0 0 0 0 0 0</pose>
         <visualize>false</visualize>
@@ -85,5 +85,5 @@
         <plugin name="gazebo_ros_laser_controller" filename="libgazebo_ros_velodyne_laser.so">
           <topicName>${topic}</topicName>
-          <frameName>${name}</frameName>
+          <frameName>/${namespace}/${name}</frameName>
           <min_range>${min_range}</min_range>
           <max_range>${max_range}</max_range>

File: velodyne_description/urdf/example.urdf.xacro (robot description, xacro)
@@ -32,7 +32,9 @@
     <origin xyz="0 0 0.4" rpy="0 0 0" />
   </VLP-16>
+<!--
   <xacro:include filename="$(find velodyne_description)/urdf/HDL-32E.urdf.xacro"/>
   <HDL-32E parent="base_link" name="velodyne2" topic="/velodyne_points2" hz="10" samples="220">
     <origin xyz="0 0 0.6" rpy="0 0 0" />
   </HDL-32E>
+-->
 </robot>
